File: DualClockLO/DualClockLO.kicad_pcb (KiCad board)
At the start: 4 copper layers, 30 x 20 mm, 23 parts, among them J1 qwiic, J2 pin header, J3 pin header, J4 pin header, J5 OEBSSEN, Y1 ECS-TX053-S3, Y3 Si5351A-B-GM

Commit message: Rev 2 modifications
Connections:
- J4 pad 2: /CLK4 -> /7/QTX
- J4 pad 3: /5/CW -> /6/ITX
- J4 pad 5: /6/ITX -> /5/CW
- J4 pad 6: /7/QTX -> /CLK4
Routing:
- net /7/QTX: track 8.71 -> 17.8 mm
- net /6/ITX: track 6.60 -> 9.19 mm, vias 0 -> 1
- net /5/CW: track 8.12 -> 6.80 mm
- net /CLK4: track 9.30 -> 10.5 mm
- net GND: vias 36 -> 33
Other:
- board text added: "Si5351A-B-GM Breakout Board Oliver King, KI3P Rev 2, 29DEC25"
- board text removed: "Si5351A-B-GM Breakout Board Oliver King, KI3P Rev 1, 25NOV25"
Changed lines of the file:
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@@
 		(tags "solder jumper open")
 		(property "Reference" "JP2"
-			(at -2.54 0 270)
+			(at -5.752001 0.127 270)
 			(layer "F.SilkS")
 			(effects
@@
 			(layers "*.Cu" "*.Mask")
 			(remove_unused_layers no)
-			(net 22 "/CLK4")
+			(net 19 "/7{slash}QTX")
 			(pinfunction "Pin_2")
 			(pintype "passive")
@@
 			(layers "*.Cu" "*.Mask")
 			(remove_unused_layers no)
-			(net 20 "/5{slash}CW")
+			(net 18 "/6{slash}ITX")
 			(pinfunction "Pin_3")
 			(pintype "passive")
@@
 			(layers "*.Cu" "*.Mask")
 			(remove_unused_layers no)
-			(net 18 "/6{slash}ITX")
+			(net 20 "/5{slash}CW")
 			(pinfunction "Pin_5")
 			(pintype "passive")
@@
 			(layers "*.Cu" "*.Mask")
 			(remove_unused_layers no)
-			(net 19 "/7{slash}QTX")
+			(net 22 "/CLK4")
 			(pinfunction "Pin_6")
 			(pintype "passive")
@@
 		(tags "net tie solder jumper bridged")
 		(property "Reference" "JP1"
-			(at 2.286 0 90)
+			(at 5.588 0.127 90)
 			(layer "F.SilkS")
 			(effects
@@
 		)
 	)
-	(gr_text "Si5351A-B-GM \nBreakout Board\nOliver King, KI3P\nRev 1, 25NOV25"
+	(gr_text "Si5351A-B-GM \nBreakout Board\nOliver King, KI3P\nRev 2, 29DEC25"
 		(at 124.714 91.948 0)
 		(layer "B.SilkS")
@@
 	)
 	(via
-		(at 118.999 91.567)
-		(size 0.6)
-		(drill 0.3)
-		(layers "F.Cu" "B.Cu")
-		(net 2)
-	)
-	(via
 		(at 125.095 93.345)
 		(size 0.6)
@@
 	)
 	(via
-		(at 116.84 91.44)
-		(size 0.6)
-		(drill 0.3)
-		(layers "F.Cu" "B.Cu")
-		(net 2)
-	)
-	(via
 		(at 139.446 91.44)
 		(size 0.6)
@@
 	)
 	(via
-		(at 116.84 93.345)
+		(at 117.5512 92.8116)
 		(size 0.6)
 		(drill 0.3)
 		(layers "F.Cu" "B.Cu")
+		(free yes)
 		(net 2)
 	)
@@
 	)
 	(via
-		(at 118.999 93.345)
-		(size 0.6)
-		(drill 0.3)
-		(layers "F.Cu" "B.Cu")
-		(net 2)
-	)
-	(via
 		(at 123.825 85.09)
 		(size 0.6)
@@
 	)
 	(segment
-		(start 118.110001 89.764999)
-		(end 118.716 89.159)
+		(start 118.716 89.159)
+		(end 118.716 91.434)
 		(width 0.2)
 		(layer "F.Cu")
@@
 	)
 	(segment
-		(start 118.110001 89.764999)
-		(end 118.11 95.504)
+		(start 118.716 91.434)
+		(end 118.3386 91.8114)
 		(width 0.2)
 		(layer "F.Cu")
 		(net 18)
 	)
+	(via
+		(at 118.3386 91.8114)
+		(size 0.6)
+		(drill 0.3)
+		(layers "F.Cu" "B.Cu")
+		(net 18)
+	)
 	(segment
-		(start 115.824 89.281)
-		(end 115.824 95.25)
+		(start 120.177 93.6498)
+		(end 121.3358 93.6498)
 		(width 0.2)
-		(layer "F.Cu")
-		(net 19)
+		(layer "B.Cu")
+		(net 18)
 	)
 	(segment
-		(start 116.896 88.209)
-		(end 117.766 88.209)
+		(start 121.3358 93.6498)
+		(end 123.19 95.504)
 		(width 0.2)
-		(layer "F.Cu")
-		(net 19)
+		(layer "B.Cu")
+		(net 18)
 	)
 	(segment
-		(start 115.824 95.25)
-		(end 115.57 95.504)
+		(start 118.3386 91.8114)
+		(end 120.177 93.6498)
+		(width 0.2)
+		(layer "B.Cu")
+		(net 18)
+	)
+	(segment
+		(start 116.789 89.186)
+		(end 116.789 95.81076)
 		(width 0.2)
 		(layer "F.Cu")
@@
 	)
 	(segment
-		(start 115.824 89.281)
-		(end 116.896 88.209)
+		(start 117.766 88.209)
+		(end 116.789 89.186)
 		(width 0.2)
 		(layer "F.Cu")
@@
 	)
 	(segment
-		(start 119.216 90.641)
-		(end 119.216 89.159)
+		(start 116.789 95.81076)
+		(end 117.63324 96.655)
 		(width 0.2)
 		(layer "F.Cu")
-		(net 20)
+		(net 19)
 	)
 	(segment
-		(start 119.8 92.339601)
-		(end 122.964399 95.504)
+		(start 117.63324 96.655)
+		(end 124.579 96.655)
 		(width 0.2)
 		(layer "F.Cu")
-		(net 20)
+		(net 19)
 	)
 	(segment
-		(start 119.8 91.225)
-		(end 119.8 92.339601)
+		(start 124.579 96.655)
+		(end 125.73 95.504)
 		(width 0.2)
 		(layer "F.Cu")
-		(net 20)
+		(net 19)
 	)
 	(segment
-		(start 122.964399 95.504)
-		(end 123.19 95.504)
+		(start 119.216 94.398)
+		(end 118.11 95.504)
 		(width 0.2)
 		(layer "F.Cu")
@@
 	)
 	(segment
-		(start 119.8 91.225)
-		(end 119.216 90.641)
+		(start 119.216 89.159)
+		(end 119.216 94.398)
 		(width 0.2)
 		(layer "F.Cu")
@@
 	)
 	(segment
-		(start 120.363303 89.978864)
-		(end 120.225864 89.978864)
+		(start 120.216 89.159)
+		(end 120.216 89.847119)
 		(width 0.2)
 		(layer "F.Cu")
@@
 	)
 	(segment
-		(start 120.216 89.969)
-		(end 120.216 89.159)
-		(width 0.2)
-		(layer "F.Cu")
-		(net 22)
-	)
-	(segment
-		(start 120.225864 89.978864)
-		(end 120.216 89.969)
+		(start 120.216 89.847119)
+		(end 120.316 89.947119)
 		(width 0.2)
 		(layer "F.Cu")
@@
 	)
 	(via
-		(at 120.363303 89.978864)
+		(at 120.316 89.947119)
 		(size 0.6)
 		(drill 0.3)
@@
 	)
 	(segment
-		(start 120.363303 89.978864)
-		(end 120.363303 91.153303)
+		(start 115.57 91.781943)
+		(end 115.57 95.504)
 		(width 0.2)
 		(layer "B.Cu")
@@
 	)
 	(segment
-		(start 124.206 93.98)
-		(end 125.73 95.504)
+		(start 120.316 90.758)
+		(end 119.8626 91.2114)
+		(width 0.2)
+		(layer "B.Cu")
+		(net 22)
+	)
+	(segment
+		(start 116.140543 91.2114)
+		(end 115.57 91.781943)
 		(width 0.2)
 		(layer "B.Cu")
@@
 	)
 	(segment
-		(start 123.19 93.98)
-		(end 124.206 93.98)
+		(start 119.8626 91.2114)
+		(end 116.140543 91.2114)
 		(width 0.2)
 		(layer "B.Cu")
@@
 	)
 	(segment
-		(start 120.363303 91.153303)
-		(end 123.19 93.98)
+		(start 120.316 89.947119)
+		(end 120.316 90.758)
 		(width 0.2)
 		(layer "B.Cu")
