File: DualClockLO/DualClockLO.kicad_sch (KiCad schematic)
At the start: 23 parts, among them J1 qwiic, J2 pin header, J3 pin header, J4 pin header, J5 OEBSSEN, Y1 ECS-TX053-S3, Y3 Si5351A-B-GM

Commit message: Rev 2 modifications
Connections:
- net 5/CW: now also J4.5 (Pin_5); no longer J4.3 (Pin_3)
- net 6/ITX: now also J4.3 (Pin_3); no longer J4.5 (Pin_5)
- net 7/QTX: now also J4.2 (Pin_2); no longer J4.6 (Pin_6)
- net CLK4: now also J4.6 (Pin_6); no longer J4.2 (Pin_2)
Other:
- moved on the sheet: J4
Changed lines of the file:
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@@
 	(title_block
 		(title "Si5351A-B-GM Breakout Board")
-		(date "2025-11-25")
-		(rev "1")
+		(date "2025-12-29")
+		(rev "2")
 		(company "Oliver King, KI3P")
 	)
@@
 	(wire
 		(pts
+			(xy 245.11 96.52) (xy 254 96.52)
+		)
+		(stroke
+			(width 0)
+			(type default)
+		)
+	)
+	(wire
+		(pts
 			(xy 222.25 90.17) (xy 243.84 90.17)
 		)
@@
 	(wire
 		(pts
-			(xy 252.73 99.06) (xy 252.73 100.33)
+			(xy 245.11 105.41) (xy 245.11 96.52)
 		)
 		(stroke
@@
 	(wire
 		(pts
+			(xy 250.19 104.14) (xy 254 104.14)
+		)
+		(stroke
+			(width 0)
+			(type default)
+		)
+	)
+	(wire
+		(pts
 			(xy 242.57 82.55) (xy 246.38 82.55)
 		)
@@
 	(wire
 		(pts
-			(xy 252.73 97.79) (xy 242.57 97.79)
-		)
-		(stroke
-			(width 0)
-			(type default)
-		)
-	)
-	(wire
-		(pts
 			(xy 201.93 50.8) (xy 201.93 69.85)
 		)
@@
 	(wire
 		(pts
-			(xy 242.57 97.79) (xy 242.57 100.33)
-		)
-		(stroke
-			(width 0)
-			(type default)
-		)
-	)
-	(wire
-		(pts
 			(xy 212.09 66.04) (xy 213.36 66.04)
 		)
@@
 	(wire
 		(pts
+			(xy 250.19 95.25) (xy 250.19 104.14)
+		)
+		(stroke
+			(width 0)
+			(type default)
+		)
+	)
+	(wire
+		(pts
 			(xy 207.01 53.34) (xy 207.01 64.77)
 		)
@@
 	(wire
 		(pts
-			(xy 245.11 102.87) (xy 245.11 105.41)
-		)
-		(stroke
-			(width 0)
-			(type default)
-		)
-	)
-	(wire
-		(pts
-			(xy 252.73 106.68) (xy 252.73 105.41)
-		)
-		(stroke
-			(width 0)
-			(type default)
-		)
-	)
-	(wire
-		(pts
-			(xy 222.25 95.25) (xy 252.73 95.25)
-		)
-		(stroke
-			(width 0)
-			(type default)
-		)
-	)
-	(wire
-		(pts
-			(xy 246.38 99.06) (xy 252.73 99.06)
-		)
-		(stroke
-			(width 0)
-			(type default)
-		)
-	)
-	(wire
-		(pts
-			(xy 252.73 102.87) (xy 245.11 102.87)
+			(xy 246.38 99.06) (xy 254 99.06)
 		)
 		(stroke
@@
 	(wire
 		(pts
-			(xy 250.19 90.17) (xy 252.73 90.17)
+			(xy 250.19 90.17) (xy 254 90.17)
 		)
 		(stroke
@@
 	(wire
 		(pts
-			(xy 222.25 100.33) (xy 242.57 100.33)
+			(xy 222.25 100.33) (xy 251.46 100.33)
 		)
 		(stroke
@@
 	(wire
 		(pts
+			(xy 222.25 95.25) (xy 250.19 95.25)
+		)
+		(stroke
+			(width 0)
+			(type default)
+		)
+	)
+	(wire
+		(pts
 			(xy 212.09 69.85) (xy 212.09 66.04)
 		)
@@
 	(wire
 		(pts
-			(xy 222.25 110.49) (xy 248.92 110.49)
+			(xy 222.25 110.49) (xy 252.73 110.49)
 		)
 		(stroke
@@
 	(wire
 		(pts
-			(xy 248.92 106.68) (xy 252.73 106.68)
+			(xy 252.73 93.98) (xy 254 93.98)
 		)
 		(stroke
@@
 	(wire
 		(pts
+			(xy 251.46 101.6) (xy 254 101.6)
+		)
+		(stroke
+			(width 0)
+			(type default)
+		)
+	)
+	(wire
+		(pts
 			(xy 137.16 80.01) (xy 133.35 80.01)
 		)
@@
 	(wire
 		(pts
+			(xy 252.73 110.49) (xy 252.73 93.98)
+		)
+		(stroke
+			(width 0)
+			(type default)
+		)
+	)
+	(wire
+		(pts
 			(xy 156.21 90.17) (xy 163.83 90.17)
 		)
@@
 	(wire
 		(pts
-			(xy 252.73 90.17) (xy 252.73 92.71)
+			(xy 254 90.17) (xy 254 91.44)
 		)
 		(stroke
@@
 	(wire
 		(pts
-			(xy 248.92 110.49) (xy 248.92 106.68)
-		)
-		(stroke
-			(width 0)
-			(type default)
-		)
-	)
-	(wire
-		(pts
 			(xy 237.49 148.59) (xy 233.68 148.59)
 		)
@@
 		(pts
 			(xy 207.01 53.34) (xy 217.17 53.34)
+		)
+		(stroke
+			(width 0)
+			(type default)
+		)
+	)
+	(wire
+		(pts
+			(xy 251.46 100.33) (xy 251.46 101.6)
 		)
 		(stroke
@@
 	(symbol
 		(lib_id "Connector:Conn_01x06_Socket")
-		(at 257.81 97.79 0)
+		(at 259.08 96.52 0)
 		(unit 1)
 		(exclude_from_sim no)
@@
 		(fields_autoplaced yes)
 		(property "Reference" "J4"
-			(at 258.5212 97.8478 0)
+			(at 259.7912 96.5778 0)
 			(effects
 				(font
@@
 		)
 		(property "Value" "pin header"
-			(at 258.5212 100.2721 0)
+			(at 259.7912 99.0021 0)
 			(effects
 				(font
@@
 		)
 		(property "Footprint" "Connector_PinHeader_2.54mm:PinHeader_1x06_P2.54mm_Vertical"
-			(at 257.81 97.79 0)
+			(at 259.08 96.52 0)
 			(effects
 				(font
@@
 		)
 		(property "Datasheet" "~"
-			(at 257.81 97.79 0)
+			(at 259.08 96.52 0)
 			(effects
 				(font
@@
 		)
 		(property "Description" "Generic connector, single row, 01x06, script generated"
-			(at 257.81 97.79 0)
-			(effects
-				(font
+			(at 259.08 96.52 0)
+			(effects
+				(font
